Commit message: update configs

File: src/vehicle_simulator/urdf/lidar.urdf.xacro (robot description, xacro)
@@ -2,5 +2,5 @@
   <link name="lidar" />
   <xacro:include filename="$(find velodyne_description)/urdf/VLP-16.urdf.xacro"/>
-  <xacro:VLP-16 parent="lidar" name="velodyne" topic="/velodyne_points" hz="5" samples="350" min_range="0.1" organize_cloud="true">
+  <xacro:VLP-16 parent="lidar" name="velodyne" topic="/velodyne_points" hz="10" samples="350" min_range="0.1" organize_cloud="true">
     <origin xyz="0 0 0" rpy="0 0 0" />
   </xacro:VLP-16>

File: src/vehicle_simulator/urdf/robot.urdf.xacro (robot description, xacro)
@@ -6,7 +6,7 @@
   </xacro:macro>
   <link name="base_origin">
-    <visual>
-      <origin xyz="0 0 0" rpy="0 0 0"/>
-    </visual>
+    <!--<visual>-->
+    <!--  <origin xyz="0 0 0" rpy="0 0 0"/>-->
+    <!--</visual>-->
   </link>
   <link name="base_link">
